File: hardware/pcb/climate_control.kicad_pcb (KiCad board)
At the start: 2 copper layers, 18 x 55 mm, 35 parts, among them J1 Switch, J2 BatteryIn, J3 USB_C, J4 HeatElement, J5 ICSP, Q2 NTR3C21NZ, U1 TP4056, U2 XB8089A, U3 ATmega328PB-AU, U4 TPS61230DRC

Commit message: Convert to Kicad 7
Connections:
- net ~RST renamed ~{RST}
Other:
- net class Default removed
